Commit message: gazebo working not aligned properly

File: description/robot.urdf.xacro (robot description, xacro)
@@ -2,3 +2,4 @@
 <robot xmlns:xacro="http://www.ros.org/wiki/xacro"  name="robot">
     <xacro:include filename="robot_core.xacro" />
+    <xacro:include filename="gazebo_control.xacro"/>
 </robot>

File: description/robot_core.xacro (robot description, xacro)
@@ -34,13 +34,15 @@
         </visual>
         <collision>
-            <origin xyz="0 0 0" rpy="0 0 0"/>
-            <geometry>
-                <box size="0.3 0.3 0.15"/>
-            </geometry>
-        </collision>
+    <origin xyz="0 0 0.08" rpy="0 0 0"/>
+    <geometry>
+        <box size="0.3 0.3 0.1"/> </geometry>
+	</collision>
         <xacro:inertial_box mass="0.5" x="0.3" y="0.3" z="0.15">
             <origin xyz="0 0 0" rpy="0 0 0"/>
         </xacro:inertial_box>
     </link>
+<gazebo reference="chassis">
+        <material>Gazebo/Blue</material>
+    </gazebo>
 <!-- REAR LEFT WHEEL -->
 <joint name="rear_left_wheel_joint" type="continuous">
@@ -64,4 +66,7 @@
             </geometry>
         </collision>
+        <xacro:inertial_cylinder mass="0.1" length="0.04" radius="0.05">
+            <origin xyz="0 0 0" rpy="0 0 0"/>
+        </xacro:inertial_cylinder>
     </link>
 <!-- FRONT LEFT WHEEL -->
@@ -86,4 +91,7 @@
             </geometry>
         </collision>
+        <xacro:inertial_cylinder mass="0.1" length="0.04" radius="0.05">
+            <origin xyz="0 0 0" rpy="0 0 0"/>
+        </xacro:inertial_cylinder>
     </link>
 <!-- FRONT RIGHT WHEEL -->
@@ -108,4 +116,7 @@
             </geometry>
         </collision>
+        <xacro:inertial_cylinder mass="0.1" length="0.04" radius="0.05">
+            <origin xyz="0 0 0" rpy="0 0 0"/>
+        </xacro:inertial_cylinder>
     </link>
 <!-- REAR RIGHT WHEEL -->
@@ -130,4 +141,7 @@
             </geometry>
         </collision>
+        <xacro:inertial_cylinder mass="0.1" length="0.04" radius="0.05">
+            <origin xyz="0 0 0" rpy="0 0 0"/>
+        </xacro:inertial_cylinder>
     </link>
 </robot>

Commit message: ros2 control pluggin and hardware interface added

File: description/robot.urdf.xacro (robot description, xacro)
@@ -1,5 +1,12 @@
 <?xml version="1.0"?>
-<robot xmlns:xacro="http://www.ros.org/wiki/xacro"  name="robot">
+<robot xmlns:xacro="http://www.ros.org/wiki/xacro" name="robot">
+    <xacro:arg name="use_mock_hardware" default="false" />
+    <xacro:arg name="use_gz_sim" default="false" />
     <xacro:include filename="robot_core.xacro" />
-    <xacro:include filename="gazebo_control.xacro"/>
+    <xacro:include filename="diffbot.ros2_control.xacro" />
+    <xacro:diffbot_ros2_control
+        name="MyBot"
+        prefix=""
+        use_mock_hardware="$(arg use_mock_hardware)"
+        use_gz_sim="$(arg use_gz_sim)"/>
 </robot>

File: description/robot_core.xacro (robot description, xacro)
@@ -18,5 +18,5 @@
         <origin xyz="0 0 0.087" rpy="0 0 0"/>
     </joint>
-<link name="chassis">
+    <link name="chassis">
         <visual>
             <origin xyz="0 0 0" rpy="0 0 0"/>
