Commit message: gazebo version updtd to 11.10

File: description/gazebo_control.xacro (robot description, xacro)
@@ -1,24 +1,27 @@
 <?xml version="1.0"?>
 <robot xmlns:xacro="http://www.ros.org/wiki/xacro">
-<gazebo>
-    <plugin name="gz::sim::systems::DiffDrive" filename="gz-sim-diff-drive-system">
-        <left_joint>front_left_wheel_joint</left_joint>
-        <left_joint>rear_left_wheel_joint</left_joint>
-        <right_joint>front_right_wheel_joint</right_joint>
-        <right_joint>rear_right_wheel_joint</right_joint>
-        <wheel_separation>0.164</wheel_separation>
-        <wheel_radius>0.04</wheel_radius> <topic>cmd_vel</topic>
-        <odom_topic>odom</odom_topic>
-        <frame_id>odom</frame_id>
-        <child_frame_id>base_link</child_frame_id>
-        <tf_topic>tf</tf_topic>
-    </plugin>
-    <plugin name="gz::sim::systems::JointStatePublisher" filename="gz-sim-joint-state-publisher-system">
-        <topic>joint_states</topic>
-        <joint_name>front_left_wheel_joint</joint_name>
-        <joint_name>rear_left_wheel_joint</joint_name>
-        <joint_name>front_right_wheel_joint</joint_name>
-        <joint_name>rear_right_wheel_joint</joint_name>
-    </plugin>
-</gazebo>
+    <gazebo>
+        <plugin name="skid_steer_drive" filename="libgazebo_ros_diff_drive.so">
+            <ros>
+                <remapping>cmd_vel:=cmd_vel</remapping>
+                <remapping>odom:=odom</remapping>
+            </ros>
+            <num_wheel_pairs>2</num_wheel_pairs>
+            <left_joint>front_left_wheel_joint</left_joint>
+            <right_joint>front_right_wheel_joint</right_joint>
+            <left_joint>rear_left_wheel_joint</left_joint>
+            <right_joint>rear_right_wheel_joint</right_joint>
+            <wheel_separation>0.35</wheel_separation>
+            <wheel_separation>0.35</wheel_separation>
+            <wheel_diameter>0.08</wheel_diameter>
+            <wheel_diameter>0.08</wheel_diameter>
+            <max_wheel_torque>20</max_wheel_torque>
+            <max_wheel_acceleration>1.0</max_wheel_acceleration>
+            <publish_odom>true</publish_odom>
+            <publish_odom_tf>true</publish_odom_tf>
+            <publish_wheel_tf>true</publish_wheel_tf>
+            <odometry_frame>odom</odometry_frame>
+            <robot_base_frame>base_link</robot_base_frame>
+        </plugin>
+    </gazebo>
 </robot>

File: description/robot.urdf.xacro (robot description, xacro)
@@ -6,4 +6,6 @@
     <xacro:include filename="robot_components.xacro" />
     <xacro:include filename="diffbot.ros2_control.xacro" />
+    <xacro:include filename="lidar.xacro" />
+    <xacro:include filename="gazebo_control.xacro" />
     <xacro:diffbot_ros2_control
         name="MyBot"

File: description/robot_components.xacro (robot description, xacro)
@@ -186,23 +186,3 @@
         <material>Gazebo/Black</material>
     </gazebo>
-	<joint name="laser_joint" type="fixed">
-        <parent link="lidar_camera_holder"/>
-        <child link="laser_frame"/>
-        <origin xyz="0 0 0" rpy="0 0 0"/> </joint>  <!--  the orientation and stl file needs to be replaced when the lidar integration happens ; like the chassis -->
-    <link name="laser_frame">
-        <visual>
-            <geometry>
-                <mesh filename="package://calixto-ros-bot/description/meshes/ROS2-Chasis-lidar-black.stl" scale="0.001 0.001 0.001"/>
-            </geometry>
-            <material name="black"/>
-        </visual>
-        <collision>
-            <geometry>
-                <cylinder radius="0.05" length="0.04"/>
-            </geometry>
-        </collision>
-        <xacro:inertial_cylinder mass="0.1" length="0.04" radius="0.05">
-            <origin xyz="0 0 0" rpy="0 0 0"/>
-        </xacro:inertial_cylinder>
-    </link>
 </robot>

File: description/robot_core.xacro (robot description, xacro)
@@ -90,5 +90,5 @@
         <parent link="base_link"/>
         <child link="front_right_wheel"/>
-        <origin xyz="0.085 -0.155 0.04" rpy="-1.5708 0 0"/> [cite: 22]
+        <origin xyz="0.085 -0.152 0.04" rpy="-1.5708 0 0"/> [cite: 22]
         <axis xyz="0 0 1"/>
     </joint>
@@ -112,5 +112,5 @@
         <parent link="base_link"/>
         <child link="rear_right_wheel"/>
-        <origin xyz="-0.085 -0.155 0.04" rpy="-1.5708 0 0"/> [cite: 23]
+        <origin xyz="-0.085 -0.152 0.04" rpy="-1.5708 0 0"/> [cite: 23]
         <axis xyz="0 0 1"/>
     </joint>
