Commit message: four wheels added ; seen with joint_state_publisher_gui

File: description/robot_core.xacro (robot description, xacro)
@@ -43,14 +43,79 @@
         </xacro:inertial_box>
     </link>
+<!-- REAR LEFT WHEEL -->
+<joint name="rear_left_wheel_joint" type="continuous">
+        <parent link="base_link"/>
+        <child link="rear_left_wheel"/>
+        <origin xyz="0.155 0.084 0.04" rpy="1.570795 0 0"/> <!-- state_publisher_gui Affects here -->
+        <axis xyz="1 0 0"/>
+    </joint>
+    <link name="rear_left_wheel">
+        <visual>
+            <geometry>
+                <mesh filename="package://my_bot/description/meshes/ROS2-wheel_FL.stl"
+                      scale="0.001 0.001 0.001"/>
+            </geometry>
+            <material name="black"/>
+        </visual>
+        <collision>
+            <origin xyz="0 0 0" rpy="1.570795 0 0"/>
+            <geometry>
+                <cylinder length="0.04" radius="0.05"/>
+            </geometry>
+        </collision>
+    </link>
 <!-- FRONT LEFT WHEEL -->
 <joint name="front_left_wheel_joint" type="continuous">
         <parent link="base_link"/>
         <child link="front_left_wheel"/>
-        <origin xyz="0.16 0 0" rpy="1.570795 0 0"/>
+        <origin xyz="0.155 -0.082 0.04" rpy="1.570795 0 0"/> <!-- state_publisher_gui Affects here -->
         <axis xyz="1 0 0"/>
     </joint>
     <link name="front_left_wheel">
         <visual>
+            <geometry>
+                <mesh filename="package://my_bot/description/meshes/ROS2-wheel_FL.stl"
+                      scale="0.001 0.001 0.001"/>
+            </geometry>
+            <material name="black"/>
+        </visual>
+        <collision>
             <origin xyz="0 0 0" rpy="1.570795 0 0"/>
+            <geometry>
+                <cylinder length="0.04" radius="0.05"/>
+            </geometry>
+        </collision>
+    </link>
+<!-- FRONT RIGHT WHEEL -->
+<joint name="front_right_wheel_joint" type="continuous">
+        <parent link="base_link"/>
+        <child link="front_right_wheel"/>
+        <origin xyz="-0.155 -0.082 0.04" rpy="0 3.14159 0"/> <!-- state_publisher_gui Affects here -->
+        <axis xyz="-1 0 0"/>
+    </joint>
+    <link name="front_right_wheel">
+        <visual>
+            <geometry>
+                <mesh filename="package://my_bot/description/meshes/ROS2-wheel_FL.stl"
+                      scale="0.001 0.001 0.001"/>
+            </geometry>
+            <material name="black"/>
+        </visual>
+        <collision>
+            <origin xyz="0 0 0" rpy="1.570795 0 0"/>
+            <geometry>
+                <cylinder length="0.04" radius="0.05"/>
+            </geometry>
+        </collision>
+    </link>
+<!-- REAR RIGHT WHEEL -->
+<joint name="rear_right_wheel_joint" type="continuous">
+        <parent link="base_link"/>
+        <child link="rear_right_wheel"/>
+        <origin xyz="-0.155 0.084 0.04" rpy="0 3.14159 0"/> <!-- state_publisher_gui Affects here -->
+        <axis xyz="-1 0 0"/>
+    </joint>
+    <link name="rear_right_wheel">
+        <visual>
             <geometry>
                 <mesh filename="package://my_bot/description/meshes/ROS2-wheel_FL.stl"

Commit message: still not stable

File: description/robot_core.xacro (robot description, xacro)
@@ -18,9 +18,14 @@
     </material>
     <link name="base_link"/>
-    <!-- CHASSIS -->
+    <!-- ═══════════════════════════════════════════════════
+         CHASSIS
+         Dimensions: L=300mm W=250mm H=120mm
+         Wheel radius = 40mm, so chassis bottom sits at Z=0.04
+         Chassis center Z = 0.04 + (0.12/2) = 0.10
+         ═══════════════════════════════════════════════════ -->
     <joint name="chassis_joint" type="fixed">
         <parent link="base_link"/>
         <child link="chassis"/>
-        <origin xyz="0 0 0"/>
+        <origin xyz="0 0 0.06"/>
     </joint>
     <link name="chassis">
@@ -34,20 +39,27 @@
         </visual>
         <collision>
-    <origin xyz="0 0 0.08" rpy="0 0 0"/>
-    <geometry>
-        <box size="0.3 0.3 0.1"/> </geometry>
-	</collision>
-        <xacro:inertial_box mass="0.5" x="0.3" y="0.3" z="0.15">
-            <origin xyz="0 0 0" rpy="0 0 0"/>
+            <origin xyz="0 0 0.06" rpy="0 0 0"/>
+            <geometry>
+                <box size="0.3 0.25 0.125"/>
+            </geometry>
+        </collision>
+        <xacro:inertial_box mass="0.5" x="0.3" y="0.25" z="0.125">
+            <origin xyz="0 0 0.06" rpy="0 0 0"/>
         </xacro:inertial_box>
     </link>
-<gazebo reference="chassis">
+    <gazebo reference="chassis">
         <material>Gazebo/Blue</material>
     </gazebo>
-<!-- REAR LEFT WHEEL -->
-<joint name="rear_left_wheel_joint" type="continuous">
+    <!-- ═══════════════════════════════════════════════════
+         WHEELS
+         Diameter = 80mm  → radius = 0.04m
+         Length   = 40mm  → 0.04m
+         Joint Z  = wheel radius = 0.04m (axle center above ground)
+         ═══════════════════════════════════════════════════ -->
+    <!-- REAR LEFT WHEEL -->
+    <joint name="rear_left_wheel_joint" type="continuous">
         <parent link="base_link"/>
         <child link="rear_left_wheel"/>
-        <origin xyz="0.155 0.084 0.04" rpy="1.570795 0 0"/> <!-- state_publisher_gui Affects here -->
+        <origin xyz="0.155 0.083 0.04" rpy="1.570795 0 0"/>
         <axis xyz="1 0 0"/>
     </joint>
@@ -61,18 +73,18 @@
         </visual>
         <collision>
-            <origin xyz="0 0 0" rpy="1.570795 0 0"/>
+            <origin xyz="0 0 0.04" rpy="1.570795 0 0"/>
             <geometry>
-                <cylinder length="0.04" radius="0.05"/>
+                <cylinder length="0.04" radius="0.04"/>
             </geometry>
         </collision>
-        <xacro:inertial_cylinder mass="0.1" length="0.04" radius="0.05">
-            <origin xyz="0 0 0" rpy="0 0 0"/>
+        <xacro:inertial_cylinder mass="0.1" length="0.04" radius="0.04">
+            <origin xyz="0 0 0.04" rpy="0 0 0"/>
         </xacro:inertial_cylinder>
     </link>
-<!-- FRONT LEFT WHEEL -->
-<joint name="front_left_wheel_joint" type="continuous">
+    <!-- FRONT LEFT WHEEL -->
+    <joint name="front_left_wheel_joint" type="continuous">
         <parent link="base_link"/>
         <child link="front_left_wheel"/>
-        <origin xyz="0.155 -0.082 0.04" rpy="1.570795 0 0"/> <!-- state_publisher_gui Affects here -->
+        <origin xyz="0.155 -0.083 0.04" rpy="1.570795 0 0"/>
         <axis xyz="1 0 0"/>
     </joint>
@@ -86,18 +98,18 @@
         </visual>
         <collision>
-            <origin xyz="0 0 0" rpy="1.570795 0 0"/>
+            <origin xyz="0 0 0.04" rpy="1.570795 0 0"/>
             <geometry>
-                <cylinder length="0.04" radius="0.05"/>
+                <cylinder length="0.04" radius="0.04"/>
             </geometry>
         </collision>
-        <xacro:inertial_cylinder mass="0.1" length="0.04" radius="0.05">
-            <origin xyz="0 0 0" rpy="0 0 0"/>
+        <xacro:inertial_cylinder mass="0.1" length="0.04" radius="0.04">
+            <origin xyz="0 0 0.04" rpy="0 0 0"/>
         </xacro:inertial_cylinder>
     </link>
-<!-- FRONT RIGHT WHEEL -->
-<joint name="front_right_wheel_joint" type="continuous">
+    <!-- FRONT RIGHT WHEEL -->
+    <joint name="front_right_wheel_joint" type="continuous">
         <parent link="base_link"/>
         <child link="front_right_wheel"/>
-        <origin xyz="-0.155 -0.082 0.04" rpy="0 3.14159 0"/> <!-- state_publisher_gui Affects here -->
+        <origin xyz="-0.155 -0.083 0.038" rpy="0 3.14159 0"/>
         <axis xyz="-1 0 0"/>
     </joint>
@@ -111,18 +123,18 @@
         </visual>
         <collision>
-            <origin xyz="0 0 0" rpy="1.570795 0 0"/>
+            <origin xyz="0 0 0.038" rpy="1.570795 0 0"/>
             <geometry>
-                <cylinder length="0.04" radius="0.05"/>
+                <cylinder length="0.04" radius="0.04"/>
             </geometry>
         </collision>
-        <xacro:inertial_cylinder mass="0.1" length="0.04" radius="0.05">
-            <origin xyz="0 0 0" rpy="0 0 0"/>
+        <xacro:inertial_cylinder mass="0.1" length="0.04" radius="0.04">
+            <origin xyz="0 0 0.038" rpy="0 0 0"/>
         </xacro:inertial_cylinder>
     </link>
-<!-- REAR RIGHT WHEEL -->
-<joint name="rear_right_wheel_joint" type="continuous">
+    <!-- REAR RIGHT WHEEL -->
+    <joint name="rear_right_wheel_joint" type="continuous">
         <parent link="base_link"/>
         <child link="rear_right_wheel"/>
-        <origin xyz="-0.155 0.084 0.04" rpy="0 3.14159 0"/> <!-- state_publisher_gui Affects here -->
+        <origin xyz="-0.155 0.083 0.038" rpy="0 3.14159 0"/>
         <axis xyz="-1 0 0"/>
     </joint>
@@ -136,11 +148,11 @@
         </visual>
         <collision>
-            <origin xyz="0 0 0" rpy="1.570795 0 0"/>
+            <origin xyz="0 0 0.038" rpy="1.570795 0 0"/>
             <geometry>
-                <cylinder length="0.04" radius="0.05"/>
+                <cylinder length="0.04" radius="0.04"/>
             </geometry>
         </collision>
-        <xacro:inertial_cylinder mass="0.1" length="0.04" radius="0.05">
-            <origin xyz="0 0 0" rpy="0 0 0"/>
+        <xacro:inertial_cylinder mass="0.1" length="0.04" radius="0.04">
+            <origin xyz="0 0 0.038" rpy="0 0 0"/>
         </xacro:inertial_cylinder>
     </link>

Commit message: urdf with box and cylinder visual;runs fine in gazebo

File: description/robot_core.xacro (robot description, xacro)
@@ -2,30 +2,22 @@
 <robot name="my_bot" xmlns:xacro="http://www.ros.org/wiki/xacro">
     <xacro:include filename="inertial_macros.xacro" />
-    <material name="white">
-        <color rgba="1 1 1 1"/>
-    </material>
-    <material name="orange">
-        <color rgba="1 0.3 0.1 1"/>
-    </material>
-    <material name="blue">
-        <color rgba="0.2 0.2 1 1"/>
-    </material>
-    <material name="black">
-        <color rgba="0 0 0 1"/>
-    </material>
-    <material name="grey">
-        <color rgba="0.5 0.5 0.5 1"/>
-    </material>
+    <material name="white">  <color rgba="1 1 1 1"/>     </material>
+    <material name="blue">   <color rgba="0.2 0.2 1 1"/> </material>
+    <material name="black">  <color rgba="0 0 0 1"/>     </material>
+    <!-- BASE LINK sits at ground level Z=0 -->
     <link name="base_link"/>
-    <!-- ═══════════════════════════════════════════════════
+    <!-- ═══════════════════════════════════════
          CHASSIS
-         Dimensions: L=300mm W=250mm H=120mm
-         Wheel radius = 40mm, so chassis bottom sits at Z=0.04
-         Chassis center Z = 0.04 + (0.12/2) = 0.10
-         ═══════════════════════════════════════════════════ -->
+         l 300 b 250 h 140
+         chassis_joint Z = 0  (base_link at ground)
+         collision Z = wheel_radius + half_height
+                     = 0.04 + 0.06 = 0.10
+         Bottom of box = 0.10 - 0.06 = 0.04  (axle plane)
+         Top of box    = 0.10 + 0.06 = 0.16
+    ═══════════════════════════════════════ -->
     <joint name="chassis_joint" type="fixed">
         <parent link="base_link"/>
         <child link="chassis"/>
-        <origin xyz="0 0 0.06"/>
+        <origin xyz="0 0 0.11" rpy="0 0 0"/>
     </joint>
     <link name="chassis">
@@ -33,17 +25,16 @@
             <origin xyz="0 0 0" rpy="0 0 0"/>
             <geometry>
-                <mesh filename="package://my_bot/description/meshes/ROS2-Chasis.stl"
-                      scale="0.001 0.001 0.001"/>
+                <box size="0.3 0.25 0.14"/>
             </geometry>
             <material name="blue"/>
         </visual>
         <collision>
-            <origin xyz="0 0 0.06" rpy="0 0 0"/>
+            <origin xyz="0 0 0" rpy="0 0 0"/>
             <geometry>
-                <box size="0.3 0.25 0.125"/>
+                <box size="0.3 0.25 0.14"/>
             </geometry>
         </collision>
-        <xacro:inertial_box mass="0.5" x="0.3" y="0.25" z="0.125">
-            <origin xyz="0 0 0.06" rpy="0 0 0"/>
+        <xacro:inertial_box mass="0.5" x="0.3" y="0.25" z="0.14">
+            <origin xyz="0 0 0" rpy="0 0 0"/>
         </xacro:inertial_box>
     </link>
@@ -51,109 +42,115 @@
         <material>Gazebo/Blue</material>
     </gazebo>
-    <!-- ═══════════════════════════════════════════════════
-         WHEELS
-         Diameter = 80mm  → radius = 0.04m
-         Length   = 40mm  → 0.04m
-         Joint Z  = wheel radius = 0.04m (axle center above ground)
-         ═══════════════════════════════════════════════════ -->
-    <!-- REAR LEFT WHEEL -->
-    <joint name="rear_left_wheel_joint" type="continuous">
-        <parent link="base_link"/>
-        <child link="rear_left_wheel"/>
-        <origin xyz="0.155 0.083 0.04" rpy="1.570795 0 0"/>
-        <axis xyz="1 0 0"/>
-    </joint>
-    <link name="rear_left_wheel">
-        <visual>
-            <geometry>
-                <mesh filename="package://my_bot/description/meshes/ROS2-wheel_FL.stl"
-                      scale="0.001 0.001 0.001"/>
-            </geometry>
-            <material name="black"/>
-        </visual>
-        <collision>
-            <origin xyz="0 0 0.04" rpy="1.570795 0 0"/>
-            <geometry>
-                <cylinder length="0.04" radius="0.04"/>
-            </geometry>
-        </collision>
-        <xacro:inertial_cylinder mass="0.1" length="0.04" radius="0.04">
-            <origin xyz="0 0 0.04" rpy="0 0 0"/>
-        </xacro:inertial_cylinder>
-    </link>
-    <!-- FRONT LEFT WHEEL -->
-    <joint name="front_left_wheel_joint" type="continuous">
-        <parent link="base_link"/>
-        <child link="front_left_wheel"/>
-        <origin xyz="0.155 -0.083 0.04" rpy="1.570795 0 0"/>
-        <axis xyz="1 0 0"/>
-    </joint>
-    <link name="front_left_wheel">
-        <visual>
-            <geometry>
-                <mesh filename="package://my_bot/description/meshes/ROS2-wheel_FL.stl"
-                      scale="0.001 0.001 0.001"/>
-            </geometry>
-            <material name="black"/>
-        </visual>
-        <collision>
-            <origin xyz="0 0 0.04" rpy="1.570795 0 0"/>
-            <geometry>
-                <cylinder length="0.04" radius="0.04"/>
-            </geometry>
-        </collision>
-        <xacro:inertial_cylinder mass="0.1" length="0.04" radius="0.04">
-            <origin xyz="0 0 0.04" rpy="0 0 0"/>
-        </xacro:inertial_cylinder>
-    </link>
-    <!-- FRONT RIGHT WHEEL -->
-    <joint name="front_right_wheel_joint" type="continuous">
-        <parent link="base_link"/>
-        <child link="front_right_wheel"/>
-        <origin xyz="-0.155 -0.083 0.038" rpy="0 3.14159 0"/>
-        <axis xyz="-1 0 0"/>
-    </joint>
-    <link name="front_right_wheel">
-        <visual>
-            <geometry>
-                <mesh filename="package://my_bot/description/meshes/ROS2-wheel_FL.stl"
-                      scale="0.001 0.001 0.001"/>
-            </geometry>
-            <material name="black"/>
-        </visual>
-        <collision>
-            <origin xyz="0 0 0.038" rpy="1.570795 0 0"/>
-            <geometry>
-                <cylinder length="0.04" radius="0.04"/>
-            </geometry>
-        </collision>
-        <xacro:inertial_cylinder mass="0.1" length="0.04" radius="0.04">
-            <origin xyz="0 0 0.038" rpy="0 0 0"/>
-        </xacro:inertial_cylinder>
-    </link>
-    <!-- REAR RIGHT WHEEL -->
-    <joint name="rear_right_wheel_joint" type="continuous">
-        <parent link="base_link"/>
-        <child link="rear_right_wheel"/>
-        <origin xyz="-0.155 0.083 0.038" rpy="0 3.14159 0"/>
-        <axis xyz="-1 0 0"/>
-    </joint>
-    <link name="rear_right_wheel">
-        <visual>
-            <geometry>
-                <mesh filename="package://my_bot/description/meshes/ROS2-wheel_FL.stl"
-                      scale="0.001 0.001 0.001"/>
-            </geometry>
-            <material name="black"/>
-        </visual>
-        <collision>
-            <origin xyz="0 0 0.038" rpy="1.570795 0 0"/>
-            <geometry>
-                <cylinder length="0.04" radius="0.04"/>
-            </geometry>
-        </collision>
-        <xacro:inertial_cylinder mass="0.1" length="0.04" radius="0.04">
-            <origin xyz="0 0 0.038" rpy="0 0 0"/>
-        </xacro:inertial_cylinder>
-    </link>
+<!-- ═══════════════════════════════════════
+FL Wheel 4cm rad 4cm length
+    ═══════════════════════════════════════ -->
+<joint name="front_left_wheel_joint" type="continuous">
+    <parent link="base_link"/>
+    <child link="front_left_wheel"/>
+    <origin xyz="0.1 0.145 0.04" rpy="-1.5708 0 0"/>
+    <axis xyz="0 0 1"/>
+</joint>
+<link name="front_left_wheel">
+    <visual>
+        <geometry>
+            <cylinder radius="0.04" length="0.04"/>
+        </geometry>
+        <material name="black"/>
+    </visual>
+    <collision>
+        <geometry>
+            <cylinder radius="0.04" length="0.04"/>
+        </geometry>
+    </collision>
+    <xacro:inertial_cylinder mass="0.1" length="0.04" radius="0.04">
+        <origin xyz="0 0 0" rpy="0 0 0"/>
+    </xacro:inertial_cylinder>
+</link>
+<gazebo reference="front_left_wheel">
+    <material>Gazebo/Black</material>
+</gazebo>
+<!-- ═══════════════════════════════════════
+RL Wheel 4cm rad 4cm length
+    ═══════════════════════════════════════ -->
+<joint name="rear_left_wheel_joint" type="continuous">
+    <parent link="base_link"/>
+    <child link="rear_left_wheel"/>
+    <origin xyz="-0.1 0.145 0.04" rpy="-1.5708 0 0"/>
+    <axis xyz="0 0 1"/>
+</joint>
+<link name="rear_left_wheel">
+    <visual>
+        <geometry>
+            <cylinder radius="0.04" length="0.04"/>
+        </geometry>
+        <material name="black"/>
+    </visual>
+    <collision>
+        <geometry>
+            <cylinder radius="0.04" length="0.04"/>
+        </geometry>
+    </collision>
+    <xacro:inertial_cylinder mass="0.1" length="0.04" radius="0.04">
+        <origin xyz="0 0 0" rpy="0 0 0"/>
+    </xacro:inertial_cylinder>
+</link>
+<gazebo reference="rear_left_wheel">
+    <material>Gazebo/Black</material>
+</gazebo>
+<!-- ═══════════════════════════════════════
+FR Wheel 4cm rad 4cm length
+    ═══════════════════════════════════════ -->
+<joint name="front_right_wheel_joint" type="continuous">
+    <parent link="base_link"/>
+    <child link="front_right_wheel"/>
+    <origin xyz="0.1 -0.145 0.04" rpy="-1.5708 0 0"/>
+    <axis xyz="0 0 1"/>
+</joint>
+<link name="front_right_wheel">
+    <visual>
+        <geometry>
+            <cylinder radius="0.04" length="0.04"/>
+        </geometry>
+        <material name="black"/>
+    </visual>
+    <collision>
+        <geometry>
+            <cylinder radius="0.04" length="0.04"/>
+        </geometry>
+    </collision>
+    <xacro:inertial_cylinder mass="0.1" length="0.04" radius="0.04">
+        <origin xyz="0 0 0" rpy="0 0 0"/>
+    </xacro:inertial_cylinder>
+</link>
+<gazebo reference="front_right_wheel">
+    <material>Gazebo/Black</material>
+</gazebo>
+<!-- ═══════════════════════════════════════
+RR Wheel 4cm rad 4cm length
+    ═══════════════════════════════════════ -->
+<joint name="rear_right_wheel_joint" type="continuous">
+    <parent link="base_link"/>
+    <child link="rear_right_wheel"/>
+    <origin xyz="-0.1 -0.145 0.04" rpy="-1.5708 0 0"/>
+    <axis xyz="0 0 1"/>
+</joint>
+<link name="rear_right_wheel">
+    <visual>
+        <geometry>
+            <cylinder radius="0.04" length="0.04"/>
+        </geometry>
+        <material name="black"/>
+    </visual>
+    <collision>
+        <geometry>
+            <cylinder radius="0.04" length="0.04"/>
+        </geometry>
+    </collision>
+    <xacro:inertial_cylinder mass="0.1" length="0.04" radius="0.04">
+        <origin xyz="0 0 0" rpy="0 0 0"/>
+    </xacro:inertial_cylinder>
+</link>
+<gazebo reference="rear_right_wheel">
+    <material>Gazebo/Black</material>
+</gazebo>
 </robot>
