Commit message: urdf with plane colours working motion

File: description/robot_core.xacro (robot description, xacro)
@@ -9,5 +9,5 @@
     <!-- ═══════════════════════════════════════
          CHASSIS
-         l 300 b 250 h 140
+         l 300 b 250 h 110
          chassis_joint Z = 0  (base_link at ground)
          collision Z = wheel_radius + half_height
@@ -19,5 +19,5 @@
         <parent link="base_link"/>
         <child link="chassis"/>
-        <origin xyz="0 0 0.11" rpy="0 0 0"/>
+        <origin xyz="0 0 0.087" rpy="0 0 0"/>
     </joint>
     <link name="chassis">
@@ -25,5 +25,5 @@
             <origin xyz="0 0 0" rpy="0 0 0"/>
             <geometry>
-                <box size="0.3 0.25 0.14"/>
+                <mesh filename="package://calixto-ros-bot/description/meshes/ROS2-Chassis-URDF.stl" scale="0.001 0.001 0.001"/>
             </geometry>
             <material name="blue"/>
@@ -32,8 +32,8 @@
             <origin xyz="0 0 0" rpy="0 0 0"/>
             <geometry>
-                <box size="0.3 0.25 0.14"/>
+                <box size="0.3 0.25 0.11"/>
             </geometry>
         </collision>
-        <xacro:inertial_box mass="0.5" x="0.3" y="0.25" z="0.14">
+        <xacro:inertial_box mass="0.5" x="0.3" y="0.25" z="0.11">
             <origin xyz="0 0 0" rpy="0 0 0"/>
         </xacro:inertial_box>
@@ -48,5 +48,5 @@
     <parent link="base_link"/>
     <child link="front_left_wheel"/>
-    <origin xyz="0.1 0.145 0.04" rpy="-1.5708 0 0"/>
+    <origin xyz="0.09 0.152 0.04" rpy="-1.5708 0 0"/>
     <axis xyz="0 0 1"/>
 </joint>
@@ -54,5 +54,5 @@
     <visual>
         <geometry>
-            <cylinder radius="0.04" length="0.04"/>
+            <mesh filename="package://calixto-ros-bot/description/meshes/ROS2-LEFT-URDF.stl" scale="0.001 0.001 0.001"/>
         </geometry>
         <material name="black"/>
@@ -76,5 +76,5 @@
     <parent link="base_link"/>
     <child link="rear_left_wheel"/>
-    <origin xyz="-0.1 0.145 0.04" rpy="-1.5708 0 0"/>
+    <origin xyz="-0.09 0.152 0.04" rpy="-1.5708 0 0"/>
     <axis xyz="0 0 1"/>
 </joint>
@@ -82,5 +82,5 @@
     <visual>
         <geometry>
-            <cylinder radius="0.04" length="0.04"/>
+            <mesh filename="package://calixto-ros-bot/description/meshes/ROS2-LEFT-URDF.stl" scale="0.001 0.001 0.001"/>
         </geometry>
         <material name="black"/>
@@ -104,5 +104,5 @@
     <parent link="base_link"/>
     <child link="front_right_wheel"/>
-    <origin xyz="0.1 -0.145 0.04" rpy="-1.5708 0 0"/>
+    <origin xyz="0.085 -0.155 0.04" rpy="-1.5708 0 0"/>
     <axis xyz="0 0 1"/>
 </joint>
@@ -110,5 +110,5 @@
     <visual>
         <geometry>
-            <cylinder radius="0.04" length="0.04"/>
+            <mesh filename="package://calixto-ros-bot/description/meshes/ROS2-RIGHT-URDF.stl" scale="0.001 0.001 0.001"/>
         </geometry>
         <material name="black"/>
@@ -132,5 +132,5 @@
     <parent link="base_link"/>
     <child link="rear_right_wheel"/>
-    <origin xyz="-0.1 -0.145 0.04" rpy="-1.5708 0 0"/>
+    <origin xyz="-0.085 -0.155 0.04" rpy="-1.5708 0 0"/>
     <axis xyz="0 0 1"/>
 </joint>
@@ -138,5 +138,5 @@
     <visual>
         <geometry>
-            <cylinder radius="0.04" length="0.04"/>
+            <mesh filename="package://calixto-ros-bot/description/meshes/ROS2-RIGHT-URDF.stl" scale="0.001 0.001 0.001"/>
         </geometry>
         <material name="black"/>

Commit message: colour sep mesh

File: description/robot_core.xacro (robot description, xacro)
@@ -2,18 +2,15 @@
 <robot name="my_bot" xmlns:xacro="http://www.ros.org/wiki/xacro">
     <xacro:include filename="inertial_macros.xacro" />
-    <material name="white">  <color rgba="1 1 1 1"/>     </material>
+    <material name="white">  <color rgba="1 1 1 1"/>      </material>
     <material name="blue">   <color rgba="0.2 0.2 1 1"/> </material>
-    <material name="black">  <color rgba="0 0 0 1"/>     </material>
-    <!-- BASE LINK sits at ground level Z=0 -->
+    <material name="black">  <color rgba="0 0 0 1"/>      </material>
+    <material name="red">    <color rgba="1 0 0 1"/>      </material>
+    <material name="green">  <color rgba="0 1 0 1"/>      </material>
+    <material name="yellow"> <color rgba="1 1 0 1"/>      </material>
+    <material name="orange"> <color rgba="1 0.5 0 1"/>   </material>
+    <material name="grey">   <color rgba="0.5 0.5 0.5 1"/></material>
+    <material name="light_blue"> <color rgba="0.6 0.8 1.0 1.0"/> </material>
+    <material name="light_grey"><color rgba="0.7 0.7 0.7 1.0"/></material>
     <link name="base_link"/>
-    <!-- ═══════════════════════════════════════
-         CHASSIS
-         l 300 b 250 h 110
-         chassis_joint Z = 0  (base_link at ground)
-         collision Z = wheel_radius + half_height
-                     = 0.04 + 0.06 = 0.10
-         Bottom of box = 0.10 - 0.06 = 0.04  (axle plane)
-         Top of box    = 0.10 + 0.06 = 0.16
-    ═══════════════════════════════════════ -->
     <joint name="chassis_joint" type="fixed">
         <parent link="base_link"/>
@@ -21,17 +18,15 @@
         <origin xyz="0 0 0.087" rpy="0 0 0"/>
     </joint>
-    <link name="chassis">
+<link name="chassis">
         <visual>
             <origin xyz="0 0 0" rpy="0 0 0"/>
             <geometry>
-                <mesh filename="package://calixto-ros-bot/description/meshes/ROS2-Chassis-URDF.stl" scale="0.001 0.001 0.001"/>
-            </geometry>
-            <material name="blue"/>
+                <mesh filename="package://calixto-ros-bot/description/meshes/ROS2-Chasis-top-and-bottom-red.stl" scale="0.001 0.001 0.001"/>
+            </geometry>
+            <material name="red"/>
         </visual>
         <collision>
             <origin xyz="0 0 0" rpy="0 0 0"/>
-            <geometry>
-                <box size="0.3 0.25 0.11"/>
-            </geometry>
+            <geometry><box size="0.3 0.25 0.11"/></geometry>
         </collision>
         <xacro:inertial_box mass="0.5" x="0.3" y="0.25" z="0.11">
@@ -40,9 +35,80 @@
     </link>
     <gazebo reference="chassis">
+        <material>Gazebo/Red</material>
+    </gazebo>
+    <joint name="battery_joint" type="fixed">
+        <parent link="chassis"/>
+        <child link="battery_holder"/>
+        <origin xyz="0 0 0"/>
+    </joint>
+    <link name="battery_holder">
+        <visual>
+            <geometry>
+                <mesh filename="package://calixto-ros-bot/description/meshes/ROS2-Chasis-battery-holder-yellow.stl" scale="0.001 0.001 0.001"/>
+            </geometry>
+            <material name="orange"/>
+        </visual>
+    </link>
+    <gazebo reference="battery_holder">
+        <material>Gazebo/Yellow</material>
+    </gazebo>
+    <joint name="comp_joint" type="fixed">
+        <parent link="chassis"/>
+        <child link="comp_parts"/>
+        <origin xyz="0 0 0"/>
+    </joint>
+    <link name="comp_parts">
+        <visual>
+            <geometry>
+                <mesh filename="package://calixto-ros-bot/description/meshes/ROS2-Chasis-comp-holder-darkblue.stl" scale="0.001 0.001 0.001"/>
+            </geometry>
+            <material name="blue"/>
+        </visual>
+        <visual>
+            <geometry>
+                <mesh filename="package://calixto-ros-bot/description/meshes/ROS2-Chasis-stem-blue.stl" scale="0.001 0.001 0.001"/>
+            </geometry>
+            <material name="light_blue"/>
+        </visual>
+    </link>
+    <gazebo reference="comp_parts">
         <material>Gazebo/Blue</material>
     </gazebo>
-<!-- ═══════════════════════════════════════
-FL Wheel 4cm rad 4cm length
-    ═══════════════════════════════════════ -->
+    <joint name="acc_joint" type="fixed">
+        <parent link="chassis"/>
+        <child link="chassis_acc"/>
+        <origin xyz="0 0 0"/>
+    </joint>
+    <link name="chassis_acc">
+        <visual> <geometry>
+                <mesh filename="package://calixto-ros-bot/description/meshes/ROS2-Chasis-led-holder-black.stl" scale="0.001 0.001 0.001"/>
+            </geometry>
+            <material name="black"/>
+        </visual>
+        <visual> <geometry>
+                <mesh filename="package://calixto-ros-bot/description/meshes/ROS2-Chasis-motors-grey.stl" scale="0.001 0.001 0.001"/>
+            </geometry>
+            <material name="light_grey"/>
+        </visual>
+    </link>
+    <gazebo reference="chassis_acc">
+        <material>Gazebo/Grey</material>
+    </gazebo>
+    <joint name="switch_holder_joint" type="fixed">
+        <parent link="chassis"/>
+        <child link="switch_holder"/>
+        <origin xyz="0 0 0" rpy="0 0 0"/>
+    </joint>
+    <link name="switch_holder">
+        <visual>
+            <geometry>
+                <mesh filename="package://calixto-ros-bot/description/meshes/ROS2-Chasis-switch-holder.stl" scale="0.001 0.001 0.001"/>
+            </geometry>
+            <material name="white"/>
+        </visual>
+    </link>
+    <gazebo reference="switch_holder">
+        <material>Gazebo/White</material>
+    </gazebo>
 <joint name="front_left_wheel_joint" type="continuous">
     <parent link="base_link"/>
@@ -70,7 +136,4 @@
     <material>Gazebo/Black</material>
 </gazebo>
-<!-- ═══════════════════════════════════════
-RL Wheel 4cm rad 4cm length
-    ═══════════════════════════════════════ -->
 <joint name="rear_left_wheel_joint" type="continuous">
     <parent link="base_link"/>
@@ -98,7 +161,4 @@
     <material>Gazebo/Black</material>
 </gazebo>
-<!-- ═══════════════════════════════════════
-FR Wheel 4cm rad 4cm length
-    ═══════════════════════════════════════ -->
 <joint name="front_right_wheel_joint" type="continuous">
     <parent link="base_link"/>
@@ -126,7 +186,4 @@
     <material>Gazebo/Black</material>
 </gazebo>
-<!-- ═══════════════════════════════════════
-RR Wheel 4cm rad 4cm length
-    ═══════════════════════════════════════ -->
 <joint name="rear_right_wheel_joint" type="continuous">
     <parent link="base_link"/>

Commit message: readme updated, minor fix

File: description/robot_core.xacro (robot description, xacro)
@@ -13,4 +13,12 @@
     <material name="light_grey"><color rgba="0.7 0.7 0.7 1.0"/></material>
     <link name="base_link"/>
+    <!-- BASE_FOOTPRINT -->
+    <joint name="base_footprint_joint" type="fixed">
+        <parent link="base_link"/>
+        <child link="base_footprint"/>
+        <origin xyz="0 0 0" rpy="0 0 0"/>
+    </joint>
+    <link name="base_footprint">
+    </link>
     <joint name="chassis_joint" type="fixed">
         <parent link="base_link"/>
