Commit message: new mesh files added; lidar needs fix

File: description/diffbot.ros2_control.xacro (robot description, xacro)
@@ -22,5 +22,5 @@
             <param name="timeout_ms">30</param>
             <param name="loop_rate">20.0</param>
-            <param name="enc_counts_per_rev">1040</param>
+            <param name="enc_counts_per_rev">850</param>
           </xacro:unless>
         </xacro:unless>

File: description/robot.urdf.xacro (robot description, xacro)
@@ -4,4 +4,5 @@
     <xacro:arg name="use_gz_sim" default="false" />
     <xacro:include filename="robot_core.xacro" />
+    <xacro:include filename="robot_components.xacro" />
     <xacro:include filename="diffbot.ros2_control.xacro" />
     <xacro:diffbot_ros2_control

File: description/robot_core.xacro (robot description, xacro)
@@ -26,4 +26,10 @@
             <material name="red"/>
         </visual>
+        <visual>
+            <geometry>
+                <mesh filename="package://calixto-ros-bot/description/meshes/ROS2-Chasis-motors-grey.stl" scale="0.001 0.001 0.001"/>
+            </geometry>
+            <material name="light_grey"/>
+        </visual>
         <collision>
             <origin xyz="0 0 0" rpy="0 0 0"/>
@@ -37,177 +43,95 @@
         <material>Gazebo/Red</material>
     </gazebo>
-    <joint name="battery_joint" type="fixed">
-        <parent link="chassis"/>
-        <child link="battery_holder"/>
-        <origin xyz="0 0 0"/>
+    <joint name="front_left_wheel_joint" type="continuous">
+        <parent link="base_link"/>
+        <child link="front_left_wheel"/>
+        <origin xyz="0.09 0.152 0.04" rpy="-1.5708 0 0"/> [cite: 19]
+        <axis xyz="0 0 1"/>
     </joint>
-    <link name="battery_holder">
+    <link name="front_left_wheel">
         <visual>
             <geometry>
-                <mesh filename="package://calixto-ros-bot/description/meshes/ROS2-Chasis-battery-holder-yellow.stl" scale="0.001 0.001 0.001"/>
-            </geometry>
-            <material name="orange"/>
-        </visual>
-    </link>
-    <gazebo reference="battery_holder">
-        <material>Gazebo/Yellow</material>
-    </gazebo>
-    <joint name="comp_joint" type="fixed">
-        <parent link="chassis"/>
-        <child link="comp_parts"/>
-        <origin xyz="0 0 0"/>
-    </joint>
-    <link name="comp_parts">
-        <visual>
-            <geometry>
-                <mesh filename="package://calixto-ros-bot/description/meshes/ROS2-Chasis-comp-holder-darkblue.stl" scale="0.001 0.001 0.001"/>
-            </geometry>
-            <material name="blue"/>
-        </visual>
-        <visual>
-            <geometry>
-                <mesh filename="package://calixto-ros-bot/description/meshes/ROS2-Chasis-stem-blue.stl" scale="0.001 0.001 0.001"/>
-            </geometry>
-            <material name="light_blue"/>
-        </visual>
-    </link>
-    <gazebo reference="comp_parts">
-        <material>Gazebo/Blue</material>
-    </gazebo>
-    <joint name="acc_joint" type="fixed">
-        <parent link="chassis"/>
-        <child link="chassis_acc"/>
-        <origin xyz="0 0 0"/>
-    </joint>
-    <link name="chassis_acc">
-        <visual> <geometry>
-                <mesh filename="package://calixto-ros-bot/description/meshes/ROS2-Chasis-led-holder-black.stl" scale="0.001 0.001 0.001"/>
+                <mesh filename="package://calixto-ros-bot/description/meshes/ROS2-LEFT-URDF.stl" scale="0.001 0.001 0.001"/>
             </geometry>
             <material name="black"/>
         </visual>
-        <visual> <geometry>
-                <mesh filename="package://calixto-ros-bot/description/meshes/ROS2-Chasis-motors-grey.stl" scale="0.001 0.001 0.001"/>
+        <collision>
+            <geometry>
+                <cylinder radius="0.04" length="0.04"/>
             </geometry>
-            <material name="light_grey"/>
-        </visual>
+        </collision>
+        <xacro:inertial_cylinder mass="0.1" length="0.04" radius="0.04">
+            <origin xyz="0 0 0" rpy="0 0 0"/>
+        </xacro:inertial_cylinder>
     </link>
-    <gazebo reference="chassis_acc">
-        <material>Gazebo/Grey</material>
-    </gazebo>
-    <joint name="switch_holder_joint" type="fixed">
-        <parent link="chassis"/>
-        <child link="switch_holder"/>
-        <origin xyz="0 0 0" rpy="0 0 0"/>
+    <joint name="rear_left_wheel_joint" type="continuous">
+        <parent link="base_link"/>
+        <child link="rear_left_wheel"/>
+        <origin xyz="-0.09 0.152 0.04" rpy="-1.5708 0 0"/> [cite: 21]
+        <axis xyz="0 0 1"/>
     </joint>
-    <link name="switch_holder">
+    <link name="rear_left_wheel">
         <visual>
             <geometry>
-                <mesh filename="package://calixto-ros-bot/description/meshes/ROS2-Chasis-switch-holder.stl" scale="0.001 0.001 0.001"/>
+                <mesh filename="package://calixto-ros-bot/description/meshes/ROS2-LEFT-URDF.stl" scale="0.001 0.001 0.001"/>
             </geometry>
-            <material name="white"/>
+            <material name="black"/>
         </visual>
+        <collision>
+            <geometry>
+                <cylinder radius="0.04" length="0.04"/>
+            </geometry>
+        </collision>
+        <xacro:inertial_cylinder mass="0.1" length="0.04" radius="0.04">
+            <origin xyz="0 0 0" rpy="0 0 0"/>
+        </xacro:inertial_cylinder>
     </link>
-    <gazebo reference="switch_holder">
-        <material>Gazebo/White</material>
-    </gazebo>
-<joint name="front_left_wheel_joint" type="continuous">
-    <parent link="base_link"/>
-    <child link="front_left_wheel"/>
-    <origin xyz="0.09 0.152 0.04" rpy="-1.5708 0 0"/>
-    <axis xyz="0 0 1"/>
-</joint>
-<link name="front_left_wheel">
-    <visual>
-        <geometry>
-            <mesh filename="package://calixto-ros-bot/description/meshes/ROS2-LEFT-URDF.stl" scale="0.001 0.001 0.001"/>
-        </geometry>
-        <material name="black"/>
-    </visual>
-    <collision>
-        <geometry>
-            <cylinder radius="0.04" length="0.04"/>
-        </geometry>
-    </collision>
-    <xacro:inertial_cylinder mass="0.1" length="0.04" radius="0.04">
-        <origin xyz="0 0 0" rpy="0 0 0"/>
-    </xacro:inertial_cylinder>
-</link>
-<gazebo reference="front_left_wheel">
-    <material>Gazebo/Black</material>
-</gazebo>
-<joint name="rear_left_wheel_joint" type="continuous">
-    <parent link="base_link"/>
-    <child link="rear_left_wheel"/>
-    <origin xyz="-0.09 0.152 0.04" rpy="-1.5708 0 0"/>
-    <axis xyz="0 0 1"/>
-</joint>
-<link name="rear_left_wheel">
-    <visual>
-        <geometry>
-            <mesh filename="package://calixto-ros-bot/description/meshes/ROS2-LEFT-URDF.stl" scale="0.001 0.001 0.001"/>
-        </geometry>
-        <material name="black"/>
-    </visual>
-    <collision>
-        <geometry>
-            <cylinder radius="0.04" length="0.04"/>
-        </geometry>
-    </collision>
-    <xacro:inertial_cylinder mass="0.1" length="0.04" radius="0.04">
-        <origin xyz="0 0 0" rpy="0 0 0"/>
-    </xacro:inertial_cylinder>
-</link>
-<gazebo reference="rear_left_wheel">
-    <material>Gazebo/Black</material>
-</gazebo>
-<joint name="front_right_wheel_joint" type="continuous">
-    <parent link="base_link"/>
-    <child link="front_right_wheel"/>
-    <origin xyz="0.085 -0.155 0.04" rpy="-1.5708 0 0"/>
-    <axis xyz="0 0 1"/>
-</joint>
-<link name="front_right_wheel">
-    <visual>
-        <geometry>
-            <mesh filename="package://calixto-ros-bot/description/meshes/ROS2-RIGHT-URDF.stl" scale="0.001 0.001 0.001"/>
-        </geometry>
-        <material name="black"/>
-    </visual>
-    <collision>
-        <geometry>
-            <cylinder radius="0.04" length="0.04"/>
-        </geometry>
-    </collision>
-    <xacro:inertial_cylinder mass="0.1" length="0.04" radius="0.04">
-        <origin xyz="0 0 0" rpy="0 0 0"/>
-    </xacro:inertial_cylinder>
-</link>
-<gazebo reference="front_right_wheel">
-    <material>Gazebo/Black</material>
-</gazebo>
-<joint name="rear_right_wheel_joint" type="continuous">
-    <parent link="base_link"/>
-    <child link="rear_right_wheel"/>
-    <origin xyz="-0.085 -0.155 0.04" rpy="-1.5708 0 0"/>
-    <axis xyz="0 0 1"/>
-</joint>
-<link name="rear_right_wheel">
-    <visual>
-        <geometry>
-            <mesh filename="package://calixto-ros-bot/description/meshes/ROS2-RIGHT-URDF.stl" scale="0.001 0.001 0.001"/>
-        </geometry>
-        <material name="black"/>
-    </visual>
-    <collision>
-        <geometry>
-            <cylinder radius="0.04" length="0.04"/>
-        </geometry>
-    </collision>
-    <xacro:inertial_cylinder mass="0.1" length="0.04" radius="0.04">
-        <origin xyz="0 0 0" rpy="0 0 0"/>
-    </xacro:inertial_cylinder>
-</link>
-<gazebo reference="rear_right_wheel">
-    <material>Gazebo/Black</material>
-</gazebo>
+    <joint name="front_right_wheel_joint" type="continuous">
+        <parent link="base_link"/>
+        <child link="front_right_wheel"/>
+        <origin xyz="0.085 -0.155 0.04" rpy="-1.5708 0 0"/> [cite: 22]
+        <axis xyz="0 0 1"/>
+    </joint>
+    <link name="front_right_wheel">
+        <visual>
+            <geometry>
+                <mesh filename="package://calixto-ros-bot/description/meshes/ROS2-RIGHT-URDF.stl" scale="0.001 0.001 0.001"/>
+            </geometry>
+            <material name="black"/>
+        </visual>
+        <collision>
+            <geometry>
+                <cylinder radius="0.04" length="0.04"/>
+            </geometry>
+        </collision>
+        <xacro:inertial_cylinder mass="0.1" length="0.04" radius="0.04">
+            <origin xyz="0 0 0" rpy="0 0 0"/>
+        </xacro:inertial_cylinder>
+    </link>
+    <joint name="rear_right_wheel_joint" type="continuous">
+        <parent link="base_link"/>
+        <child link="rear_right_wheel"/>
+        <origin xyz="-0.085 -0.155 0.04" rpy="-1.5708 0 0"/> [cite: 23]
+        <axis xyz="0 0 1"/>
+    </joint>
+    <link name="rear_right_wheel">
+        <visual>
+            <geometry>
+                <mesh filename="package://calixto-ros-bot/description/meshes/ROS2-RIGHT-URDF.stl" scale="0.001 0.001 0.001"/>
+            </geometry>
+            <material name="black"/>
+        </visual>
+        <collision>
+            <geometry>
+                <cylinder radius="0.04" length="0.04"/>
+            </geometry>
+        </collision>
+        <xacro:inertial_cylinder mass="0.1" length="0.04" radius="0.04">
+            <origin xyz="0 0 0" rpy="0 0 0"/>
+        </xacro:inertial_cylinder>
+    </link>
+    <gazebo reference="front_left_wheel"> <material>Gazebo/Black</material> </gazebo>
+    <gazebo reference="rear_left_wheel">  <material>Gazebo/Black</material> </gazebo>
+    <gazebo reference="front_right_wheel"> <material>Gazebo/Black</material> </gazebo>
+    <gazebo reference="rear_right_wheel">  <material>Gazebo/Black</material> </gazebo>
 </robot>

Commit message: checkpoint, sim works correctly around corener with nav2 and smacd

File: description/diffbot.ros2_control.xacro (robot description, xacro)
@@ -18,5 +18,5 @@
             <param name="rear_left_wheel_name">${prefix}rear_left_wheel_joint</param>
             <param name="rear_right_wheel_name">${prefix}rear_right_wheel_joint</param>
-            <param name="device">/dev/ttyUSB0</param>
+            <param name="device">/dev/ttyLP2</param>
             <param name="baud_rate">115200</param>
             <param name="timeout_ms">30</param>

File: description/robot_core.xacro (robot description, xacro)
@@ -12,12 +12,5 @@
     <material name="light_blue"> <color rgba="0.6 0.8 1.0 1.0"/> </material>
     <material name="light_grey"><color rgba="0.7 0.7 0.7 1.0"/></material>
-    <link name="base_link"/>
-    <!-- BASE_FOOTPRINT -->
-    <joint name="base_footprint_joint" type="fixed">
-        <parent link="base_link"/>
-        <child link="base_footprint"/>
-        <origin xyz="0 0 0" rpy="0 0 0"/>
-    </joint>
-    <link name="base_footprint">
+    <link name="base_link">
     </link>
     <joint name="chassis_joint" type="fixed">
@@ -44,5 +37,5 @@
             <geometry><box size="0.3 0.25 0.11"/></geometry>
         </collision>
-        <xacro:inertial_box mass="0.5" x="0.3" y="0.25" z="0.11">
+        <xacro:inertial_box mass="2.0" x="0.3" y="0.25" z="0.11">
             <origin xyz="0 0 0" rpy="0 0 0"/>
         </xacro:inertial_box>
@@ -139,4 +132,10 @@
         </xacro:inertial_cylinder>
     </link>
+	<link name="imu_link"/>
+	<joint name="imu_joint" type="fixed">
+	  <parent link="base_link"/>
+	  <child link="imu_link"/>
+	  <origin xyz="0 0 0" rpy="0 0 0"/>
+	</joint>
     <gazebo reference="front_left_wheel"> <material>Gazebo/Black</material> </gazebo>
     <gazebo reference="rear_left_wheel">  <material>Gazebo/Black</material> </gazebo>
